File: Electronics/EAGLE/Slutsteg.brd (EAGLE design)
At the start: 100 x 160 mm, 152 parts, among them CN1 OSTYK33102030-2, CN2 OSTYK33102030-2, CN3 OSTYK33102030-2, IC1 SPX1117M3-L-3-3_TR, IC10 LM324D, IC11 L78M12ABDT-TR, IC3 ESP32-WROVER-IE-4MB, IC4 TM8211, IC6 TPA3244DDWR, IC7 TPA3251D2DDVR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

Commit message: fixade lite graj
Parts:
- C46, C50: device rcl:C1206 -> rcl:C0805
- R1, R10, R11, R2, R3, R4, R5, R6, R7, R8, R9: value 10k/5%/0.1W -> 10K/5%/0.1W
Changed lines of the file:
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@@
 <attribute name="VALUE" x="115.27" y="24.46" size="1.27" layer="27"/>
 </element>
-<element name="C50" library="rcl" library_urn="urn:adsk.eagle:library:334" package="C1206" package3d_urn="urn:adsk.eagle:package:23618/2" value="10uF/16V" x="116.54" y="20.65" smashed="yes">
+<element name="C50" library="rcl" library_urn="urn:adsk.eagle:library:334" package="C0805" package3d_urn="urn:adsk.eagle:package:23617/2" value="10uF/16V" x="116.54" y="20.65" smashed="yes">
 <attribute name="NAME" x="115.27" y="21.92" size="1.27" layer="25"/>
-<attribute name="POPULARITY" value="54" x="116.54" y="20.65" size="1.778" layer="27" display="off"/>
+<attribute name="POPULARITY" value="88" x="116.54" y="20.65" size="1.778" layer="27" display="off"/>
 <attribute name="SPICEPREFIX" value="C" x="116.54" y="20.65" size="1.778" layer="27" display="off"/>
 <attribute name="VALUE" x="115.27" y="18.11" size="1.27" layer="27"/>
 </element>
-<element name="C46" library="rcl" library_urn="urn:adsk.eagle:library:334" package="C1206" package3d_urn="urn:adsk.eagle:package:23618/2" value="10uF/16V" x="116.54" y="14.3" smashed="yes">
+<element name="C46" library="rcl" library_urn="urn:adsk.eagle:library:334" package="C0805" package3d_urn="urn:adsk.eagle:package:23617/2" value="10uF/16V" x="116.54" y="14.3" smashed="yes">
 <attribute name="NAME" x="115.27" y="15.57" size="1.27" layer="25"/>
-<attribute name="POPULARITY" value="54" x="116.54" y="14.3" size="1.778" layer="27" display="off"/>
+<attribute name="POPULARITY" value="88" x="116.54" y="14.3" size="1.778" layer="27" display="off"/>
 <attribute name="SPICEPREFIX" value="C" x="116.54" y="14.3" size="1.778" layer="27" display="off"/>
 <attribute name="VALUE" x="115.27" y="11.76" size="1.27" layer="27"/>
@@
 <attribute name="VALUE" x="-205.56" y="146.59" size="1.27" layer="27"/>
 </element>
-<element name="R6" library="rcl" library_urn="urn:adsk.eagle:library:334" package="R0603" package3d_urn="urn:adsk.eagle:package:23555/3" value="10k/5%/0.1W" x="-206.83" y="136.43" smashed="yes">
+<element name="R6" library="rcl" library_urn="urn:adsk.eagle:library:334" package="R0603" package3d_urn="urn:adsk.eagle:package:23555/3" value="10K/5%/0.1W" x="-206.83" y="136.43" smashed="yes">
 <attribute name="NAME" x="-207.465" y="137.065" size="1.27" layer="25"/>
 <attribute name="POPULARITY" value="70" x="-206.83" y="136.43" size="1.778" layer="27" display="off"/>
@@
 <attribute name="VALUE" x="-207.465" y="134.525" size="1.27" layer="27"/>
 </element>
-<element name="R8" library="rcl" library_urn="urn:adsk.eagle:library:334" package="R0603" package3d_urn="urn:adsk.eagle:package:23555/3" value="10k/5%/0.1W" x="-206.83" y="131.35" smashed="yes">
+<element name="R8" library="rcl" library_urn="urn:adsk.eagle:library:334" package="R0603" package3d_urn="urn:adsk.eagle:package:23555/3" value="10K/5%/0.1W" x="-206.83" y="131.35" smashed="yes">
 <attribute name="NAME" x="-207.465" y="131.985" size="1.27" layer="25"/>
 <attribute name="POPULARITY" value="70" x="-206.83" y="131.35" size="1.778" layer="27" display="off"/>
@@
 <attribute name="VALUE" x="-207.465" y="104.045" size="1.27" layer="27"/>
 </element>
-<element name="R9" library="rcl" library_urn="urn:adsk.eagle:library:334" package="R0603" package3d_urn="urn:adsk.eagle:package:23555/3" value="10k/5%/0.1W" x="-206.83" y="100.87" smashed="yes">
+<element name="R9" library="rcl" library_urn="urn:adsk.eagle:library:334" package="R0603" package3d_urn="urn:adsk.eagle:package:23555/3" value="10K/5%/0.1W" x="-206.83" y="100.87" smashed="yes">
 <attribute name="NAME" x="-207.465" y="101.505" size="1.27" layer="25"/>
 <attribute name="POPULARITY" value="70" x="-206.83" y="100.87" size="1.778" layer="27" display="off"/>
@@
 <attribute name="VALUE" x="-207.465" y="98.965" size="1.27" layer="27"/>
 </element>
-<element name="R11" library="rcl" library_urn="urn:adsk.eagle:library:334" package="R0603" package3d_urn="urn:adsk.eagle:package:23555/3" value="10k/5%/0.1W" x="-206.83" y="95.79" smashed="yes">
+<element name="R11" library="rcl" library_urn="urn:adsk.eagle:library:334" package="R0603" package3d_urn="urn:adsk.eagle:package:23555/3" value="10K/5%/0.1W" x="-206.83" y="95.79" smashed="yes">
 <attribute name="NAME" x="-207.465" y="96.425" size="1.27" layer="25"/>
 <attribute name="POPULARITY" value="70" x="-206.83" y="95.79" size="1.778" layer="27" display="off"/>
@@
 <attribute name="VALUE" x="-207.465" y="88.805" size="1.27" layer="27"/>
 </element>
-<element name="R1" library="rcl" library_urn="urn:adsk.eagle:library:334" package="R0603" package3d_urn="urn:adsk.eagle:package:23555/3" value="10k/5%/0.1W" x="-206.83" y="85.63" smashed="yes">
+<element name="R1" library="rcl" library_urn="urn:adsk.eagle:library:334" package="R0603" package3d_urn="urn:adsk.eagle:package:23555/3" value="10K/5%/0.1W" x="-206.83" y="85.63" smashed="yes">
 <attribute name="NAME" x="-207.465" y="86.265" size="1.27" layer="25"/>
 <attribute name="POPULARITY" value="70" x="-206.83" y="85.63" size="1.778" layer="27" display="off"/>
@@
 <attribute name="VALUE" x="-207.465" y="83.725" size="1.27" layer="27"/>
 </element>
-<element name="R7" library="rcl" library_urn="urn:adsk.eagle:library:334" package="R0603" package3d_urn="urn:adsk.eagle:package:23555/3" value="10k/5%/0.1W" x="-206.83" y="80.55" smashed="yes">
+<element name="R7" library="rcl" library_urn="urn:adsk.eagle:library:334" package="R0603" package3d_urn="urn:adsk.eagle:package:23555/3" value="10K/5%/0.1W" x="-206.83" y="80.55" smashed="yes">
 <attribute name="NAME" x="-207.465" y="81.185" size="1.27" layer="25"/>
 <attribute name="POPULARITY" value="70" x="-206.83" y="80.55" size="1.778" layer="27" display="off"/>
@@
 <attribute name="VALUE" x="-207.465" y="78.645" size="1.27" layer="27"/>
 </element>
-<element name="R10" library="rcl" library_urn="urn:adsk.eagle:library:334" package="R0603" package3d_urn="urn:adsk.eagle:package:23555/3" value="10k/5%/0.1W" x="-206.83" y="75.47" smashed="yes">
+<element name="R10" library="rcl" library_urn="urn:adsk.eagle:library:334" package="R0603" package3d_urn="urn:adsk.eagle:package:23555/3" value="10K/5%/0.1W" x="-206.83" y="75.47" smashed="yes">
 <attribute name="NAME" x="-207.465" y="76.105" size="1.27" layer="25"/>
 <attribute name="POPULARITY" value="70" x="-206.83" y="75.47" size="1.778" layer="27" display="off"/>
@@
 <attribute name="VALUE" x="-207.465" y="73.565" size="1.27" layer="27"/>
 </element>
-<element name="R2" library="rcl" library_urn="urn:adsk.eagle:library:334" package="R0603" package3d_urn="urn:adsk.eagle:package:23555/3" value="10k/5%/0.1W" x="-206.83" y="70.39" smashed="yes">
+<element name="R2" library="rcl" library_urn="urn:adsk.eagle:library:334" package="R0603" package3d_urn="urn:adsk.eagle:package:23555/3" value="10K/5%/0.1W" x="-206.83" y="70.39" smashed="yes">
 <attribute name="NAME" x="-207.465" y="71.025" size="1.27" layer="25"/>
 <attribute name="POPULARITY" value="70" x="-206.83" y="70.39" size="1.778" layer="27" display="off"/>
@@
 <attribute name="VALUE" x="-207.465" y="68.485" size="1.27" layer="27"/>
 </element>
-<element name="R3" library="rcl" library_urn="urn:adsk.eagle:library:334" package="R0603" package3d_urn="urn:adsk.eagle:package:23555/3" value="10k/5%/0.1W" x="-206.83" y="65.31" smashed="yes">
+<element name="R3" library="rcl" library_urn="urn:adsk.eagle:library:334" package="R0603" package3d_urn="urn:adsk.eagle:package:23555/3" value="10K/5%/0.1W" x="-206.83" y="65.31" smashed="yes">
 <attribute name="NAME" x="-207.465" y="65.945" size="1.27" layer="25"/>
 <attribute name="POPULARITY" value="70" x="-206.83" y="65.31" size="1.778" layer="27" display="off"/>
@@
 <attribute name="VALUE" x="-207.465" y="63.405" size="1.27" layer="27"/>
 </element>
-<element name="R4" library="rcl" library_urn="urn:adsk.eagle:library:334" package="R0603" package3d_urn="urn:adsk.eagle:package:23555/3" value="10k/5%/0.1W" x="-206.83" y="60.23" smashed="yes">
+<element name="R4" library="rcl" library_urn="urn:adsk.eagle:library:334" package="R0603" package3d_urn="urn:adsk.eagle:package:23555/3" value="10K/5%/0.1W" x="-206.83" y="60.23" smashed="yes">
 <attribute name="NAME" x="-207.465" y="60.865" size="1.27" layer="25"/>
 <attribute name="POPULARITY" value="70" x="-206.83" y="60.23" size="1.778" layer="27" display="off"/>
@@
 <attribute name="VALUE" x="-207.465" y="58.325" size="1.27" layer="27"/>
 </element>
-<element name="R5" library="rcl" library_urn="urn:adsk.eagle:library:334" package="R0603" package3d_urn="urn:adsk.eagle:package:23555/3" value="10k/5%/0.1W" x="-206.83" y="55.15" smashed="yes">
+<element name="R5" library="rcl" library_urn="urn:adsk.eagle:library:334" package="R0603" package3d_urn="urn:adsk.eagle:package:23555/3" value="10K/5%/0.1W" x="-206.83" y="55.15" smashed="yes">
 <attribute name="NAME" x="-207.465" y="55.785" size="1.27" layer="25"/>
 <attribute name="POPULARITY" value="70" x="-206.83" y="55.15" size="1.778" layer="27" display="off"/>
@@
 <contactref element="IC7" pad="5"/>
 <contactref element="C46" pad="1"/>
-<wire x1="135.612" y1="201.308" x2="115.14" y2="14.3" width="0" layer="19" extent="1-1"/>
+<wire x1="135.612" y1="201.308" x2="115.59" y2="14.3" width="0" layer="19" extent="1-1"/>
 </signal>
 <signal name="N$28">
 <contactref element="IC7" pad="6"/>
 <contactref element="C50" pad="1"/>
-<wire x1="135.612" y1="200.672" x2="115.14" y2="20.65" width="0" layer="19" extent="1-1"/>
+<wire x1="135.612" y1="200.672" x2="115.59" y2="20.65" width="0" layer="19" extent="1-1"/>
 </signal>
 <signal name="N$29">

Commit message: Börjat med TPA3251s del av kretskortet
Parts:
- moved C63 225.3 mm to (38.0, 40.7)
- moved C64 222.0 mm to (37.9, 25.7)
- moved L8 213.8 mm to (55.1, 11.2)
- moved C65 211.9 mm to (65.9, 26.9)
- moved L7 211.3 mm to (55.1, 25.3)
- moved IC7 198.6 mm to (27.4, 33.2)
- moved C66 186.1 mm to (81.0, 39.3), turned to 180 degrees
- moved C70 148.8 mm to (81.9, 10.2), turned to 90 degrees
- moved L6 145.2 mm to (55.1, 41.0)
- moved R27 143.4 mm to (84.0, 10.2), turned to 90 degrees
- moved L5 143.2 mm to (55.1, 55.0)
- moved C45 131.0 mm to (-13.5, 17.4)
- moved C46 131.0 mm to (-13.5, -1.70)
- moved C48 131.0 mm to (-13.5, 11.0)
- moved C49 131.0 mm to (-14.7, 23.7)
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Routing:
- net SPEAKER_B_1: track 0.00 -> 5.74 mm
- net SPEAKER_B_0: track 0.00 -> 4.05 mm
- net N$2: track 0.00 -> 2.08 mm
- net N$38: track 0.00 -> 2.07 mm
- added copper zone on layer 1, net N$18
- added copper zone on layer 16, net N$18
- added copper zone on layer 1, net N$19
- added copper zone on layer 1, net N$26
- added copper zone on layer 1, net N$36
- added copper zone on layer 16, net N$36
- added copper zone on layer 1, net SPEAKER_B_0
- added copper zone on layer 1, net SPEAKER_B_1
- added copper zone on layer 16, net SPEAKER_B_1

Commit message: Lagt till double-gang pot och petat lite i layouten
Parts:
- removed SW1, SW2: PDB181-K420F-103A2, PDB181-K420F-103A2:SW_420F-103A2_BRN
- added R46: PDB182-K430K-503A, Pot-PDB18:PDB18-2
- moved R45 387.3 mm to (46.0, 144.0)
- moved J2 352.3 mm to (34.0, 153.0), turned to 270 degrees
- moved SW3 345.9 mm to (7.44, 149.0), turned to 270 degrees
- moved C1 343.1 mm to (135.4, 132.7)
- moved C2 343.1 mm to (135.4, 127.6)
- moved C3 343.1 mm to (136.7, 151.8)
- moved C7 343.1 mm to (136.7, 139.1)
- moved C78 340.4 mm to (39.0, 144.0), turned to 90 degrees
- moved R10 330.3 mm to (122.2, 46.5)
- moved C79 328.7 mm to (34.0, 125.0)
- moved C25 328.3 mm to (29.0, 144.0), turned to 90 degrees
- moved C14 328.2 mm to (121.2, 102.7)
- moved R1 328.2 mm to (121.2, 97.6)
- moved R2 328.2 mm to (121.2, 82.4)
- moved R3 328.2 mm to (121.2, 77.3)
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Connections:
- net LEFT_OUT: now also R46.2, R46.3; no longer SW1.2, SW1.3
- net N$71: now also R46.1; no longer SW1.1
- net N$74: now also R46.4; no longer SW2.1
- net RIGHT_OUT: now also R46.5, R46.6; no longer SW2.2, SW2.3
Other:
- outline, holes or cut-outs redrawn
